Commit message: Camera Joint Changed

File: chessbot_ws/src/chessbot_robot/urdf/robot/joints.xacro (robot description, xacro)
@@ -57,5 +57,5 @@
     <parent link="link_6"/>
     <child link="camera_link"/>
-    <origin rpy="0 0.85 0" xyz="0.01 0 0"/>
+    <origin rpy="0 1 0" xyz="0.01 0 -0.1"/>
   </joint>
     <!-- end of joint list -->
