Commit message: Robot Definition Update. Breakdown in Links and Joints. No Macro.

File: chessbot_ws/src/chessbot_robot/urdf/irb140.xacro (robot description, xacro)
@@ -1,6 +1,8 @@
 <?xml version="1.0" ?>
 <robot name="abb_irb140" xmlns:xacro="http://ros.org/wiki/xacro">
-	<xacro:include filename="$(find chessbot_robot)/urdf/irb140_macro.xacro"/>
-	<xacro:include filename="$(find chessbot_robot)/urdf/irb140.gazebo"/>
-	<xacro:abb_irb140 prefix=""/>
+	<xacro:include filename="$(find chessbot_robot)/urdf/robot/irb140_robot.xacro"/>
+	<xacro:include filename="$(find chessbot_robot)/urdf/gazebo/camera_sensor.gazebo"/>
+	<gazebo>
+    	<static>true</static>
+	</gazebo>
 </robot>

File: chessbot_ws/src/chessbot_robot/urdf/robot/links.xacro (robot description, xacro)
@@ -1,16 +1,7 @@
-<?xml version="1.0" ?>
-<!-- =================================================================================== -->
-<!-- |    This document was autogenerated by xacro from /Users/amorales/Documents/IEEE/2022/RAS/chessbot/chessbot/chessbot_ws/src/chessbot_robot/urdf/irb140.xacro | -->
-<!-- |    EDITING THIS FILE BY HAND IS NOT RECOMMENDED                                 | -->
-<!-- =================================================================================== -->
-<robot name="abb_irb140">
-      <material name="abb_orange">
-        <color rgba="1 0.43 0 1"/>
-      </material>
-      <material name="yellow">
-        <color rgba="0 1 1 1"/>
-      </material>
-  <!-- link list -->
-  <link name="base_link">
+<?xml version="1.0"?>
+<robot>
+     <link name="world"/>
+    <!-- link list -->
+    <link name="base_link">
     <visual>
       <origin rpy="0 0 0" xyz="0 0 0"/>
@@ -18,5 +9,7 @@
         <mesh filename="package://chessbot_robot/meshes/irb140/visual/base_link.stl" scale="0.01 0.01 0.01"/>
       </geometry>
-      <material name="abb_orange"/>
+      <material name="abb_orange">
+        <color rgba="1 0.43 0 1"/>
+      </material>
     </visual>
     <collision>
@@ -24,6 +17,13 @@
         <mesh filename="package://chessbot_robot/meshes/irb140/collision/base_link.stl" scale="0.01 0.01 0.01"/>
       </geometry>
-      <material name="yellow"/>
+      <material name="yellow">
+        <color rgba="0 1 1 1"/>
+      </material>
     </collision>
+    <inertial>
+      <origin xyz="0.0 0.0 0.0" rpy="0.0 0.0 0.0"/>
+      <mass value="1.0"/>
+      <inertia ixx="0.0" ixy="0.0" ixz="0.0" iyy="0.0" iyz="0.0" izz="0.0"/>
+    </inertial>
   </link>
   <link name="link_1">
@@ -42,4 +42,9 @@
       <material name="yellow"/>
     </collision>
+     <inertial>
+      <origin xyz="0.0 0.0 0.0" rpy="0.0 0.0 0.0"/>
+      <mass value="1.0"/>
+      <inertia ixx="0.0" ixy="0.0" ixz="0.0" iyy="0.0" iyz="0.0" izz="0.0"/>
+    </inertial>
   </link>
   <link name="link_2">
@@ -58,4 +63,9 @@
       <material name="yellow"/>
     </collision>
+     <inertial>
+      <origin xyz="0.0 0.0 0.0" rpy="0.0 0.0 0.0"/>
+      <mass value="1.0"/>
+      <inertia ixx="0.0" ixy="0.0" ixz="0.0" iyy="0.0" iyz="0.0" izz="0.0"/>
+    </inertial>
   </link>
   <link name="link_3">
@@ -74,4 +84,9 @@
       <material name="yellow"/>
     </collision>
+     <inertial>
+      <origin xyz="0.0 0.0 0.0" rpy="0.0 0.0 0.0"/>
+      <mass value="1.0"/>
+      <inertia ixx="0.0" ixy="0.0" ixz="0.0" iyy="0.0" iyz="0.0" izz="0.0"/>
+    </inertial>
   </link>
   <link name="link_4">
@@ -90,4 +105,9 @@
       <material name="yellow"/>
     </collision>
+     <inertial>
+      <origin xyz="0.0 0.0 0.0" rpy="0.0 0.0 0.0"/>
+      <mass value="1.0"/>
+      <inertia ixx="0.0" ixy="0.0" ixz="0.0" iyy="0.0" iyz="0.0" izz="0.0"/>
+    </inertial>
   </link>
   <link name="link_5">
@@ -106,4 +126,9 @@
       <material name="yellow"/>
     </collision>
+     <inertial>
+      <origin xyz="0.0 0.0 0.0" rpy="0.0 0.0 0.0"/>
+      <mass value="1.0"/>
+      <inertia ixx="0.0" ixy="0.0" ixz="0.0" iyy="0.0" iyz="0.0" izz="0.0"/>
+    </inertial>
   </link>
   <link name="link_6">
@@ -122,62 +147,33 @@
       <material name="yellow"/>
     </collision>
+     <inertial>
+      <origin xyz="0.0 0.0 0.0" rpy="0.0 0.0 0.0"/>
+      <mass value="1.0"/>
+      <inertia ixx="0.0" ixy="0.0" ixz="0.0" iyy="0.0" iyz="0.0" izz="0.0"/>
+    </inertial>
   </link>
-  <link name="tool0"/>
-  <!-- end of link list -->
-  <!-- joint list -->
-  <joint name="joint_1" type="revolute">
-    <origin rpy="0 0 0" xyz="0 0 0"/>
-    <parent link="base_link"/>
-    <child link="link_1"/>
-    <axis xyz="0 0 1"/>
-    <limit effort="0" lower="-3.1416" upper="3.1416" velocity="2.618"/>
-  </joint>
-  <joint name="joint_2" type="revolute">
-    <origin rpy="0 0 0" xyz="0.070 0 0.352"/>
-    <parent link="link_1"/>
-    <child link="link_2"/>
-    <axis xyz="0 1 0"/>
-    <limit effort="0" lower="-1.7453" upper="1.7453" velocity="2.618"/>
-  </joint>
-  <joint name="joint_3" type="revolute">
-    <origin rpy="0 0 0" xyz="0 -0.065 0.360"/>
-    <parent link="link_2"/>
-    <child link="link_3"/>
-    <axis xyz="0 1 0"/>
-    <limit effort="0" lower="-2.4434" upper="2.4434" velocity="2.618"/>
-  </joint>
-  <joint name="joint_4" type="revolute">
-    <origin rpy="0 0 0" xyz="0.239 0.065 0"/>
-    <parent link="link_3"/>
-    <child link="link_4"/>
-    <axis xyz="1 0 0"/>
-    <limit effort="0" lower="-3.49" upper="3.49" velocity="6.2832"/>
-  </joint>
-  <joint name="joint_5" type="revolute">
-    <origin rpy="0 0 0" xyz="0.141 0 0"/>
-    <parent link="link_4"/>
-    <child link="link_5"/>
-    <axis xyz="0 1 0"/>
-    <limit effort="0" lower="-2.0071" upper="2.0071" velocity="6.2832"/>
-  </joint>
-  <joint name="joint_6" type="revolute">
-    <origin rpy="0 0 0" xyz="0.065 0 0"/>
-    <parent link="link_5"/>
-    <child link="link_6"/>
-    <axis xyz="1 0 0"/>
-    <limit effort="0" lower="-6.9813" upper="6.9813" velocity="7.854"/>
-  </joint>
-  <joint name="joint_6-tool0" type="fixed">
-    <parent link="link_6"/>
-    <child link="tool0"/>
-    <origin rpy="0 0 0" xyz="0 0 0"/>
-  </joint>
-  <!-- end of joint list -->
-  <!-- ROS base_link to ABB World Coordinates transform -->
-  <link name="base"/>
-  <joint name="base_link-base" type="fixed">
-    <origin rpy="0 0 0" xyz="0 0 0"/>
-    <parent link="base_link"/>
-    <child link="base"/>
-  </joint>
+  <link name="camera_link">
+    <inertial>
+      <origin xyz="0.0 0.0 0.0" rpy="0.0 0.0 0.0"/>
+      <mass value="0.0"/>
+      <inertia ixx="0.0" ixy="0.0" ixz="0.0" iyy="0.0" iyz="0.0" izz="0.0"/>
+    </inertial>
+    <visual name="">
+      <origin xyz="0.0 0.0 0.0" rpy="0.0 0.0 0.0"/>
+      <geometry>
+        <box size="0.1 0.1 0.1"/>
+      </geometry>
+      <material name="">
+        <color rgba="1.0 0.0 0.0 1.0"/>
+        <texture filename=""/>
+      </material>
+    </visual>
+    <collision>
+      <origin xyz="0.0 0.0 0.0" rpy="0.0 0.0 0.0"/>
+      <geometry>
+        <box size="0.0 0.0 0.0"/>
+      </geometry>
+    </collision>
+  </link>
+  <link name="tool0" />
 </robot>

File: chessbot_ws/src/chessbot_robot/urdf/urdf_build/irb140.urdf (robot description, URDF)
Before this commit: robot None, 0 links, 0 joints
Links:
- added link base
- added link base_link, mass 1.0; collision mesh filename=package://chessbot_robot/meshes/irb140/collision/base_link.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 scale=0.01 0.01 0.01; visual mesh filename=package://chessbot_robot/meshes/irb140/visual/base_link.stl scale=0.01 0.01 0.01
- added link camera_link, mass 0.0; collision box size=0.0 0.0 0.0; visual box size=0.1 0.1 0.1
- added link link_1, mass 1.0; collision mesh filename=package://chessbot_robot/meshes/irb140/collision/link_1.stl scale=0.01 0.01 0.01; visual mesh filename=package://chessbot_robot/meshes/irb140/visual/link_1.stl scale=0.01 0.01 0.01
- added link link_2, mass 1.0; collision mesh filename=package://chessbot_robot/meshes/irb140/collision/link_2.stl scale=0.01 0.01 0.01; visual mesh filename=package://chessbot_robot/meshes/irb140/visual/link_2.stl scale=0.01 0.01 0.01
- added link link_3, mass 1.0; collision mesh filename=package://chessbot_robot/meshes/irb140/collision/link_3.stl scale=0.01 0.01 0.01; visual mesh filename=package://chessbot_robot/meshes/irb140/visual/link_3.stl scale=0.01 0.01 0.01
- added link link_4, mass 1.0; collision mesh filename=package://chessbot_robot/meshes/irb140/collision/link_4.stl scale=0.01 0.01 0.01; visual mesh filename=package://chessbot_robot/meshes/irb140/visual/link_4.stl scale=0.01 0.01 0.01
- added link link_5, mass 1.0; collision mesh filename=package://chessbot_robot/meshes/irb140/collision/link_5.stl scale=0.01 0.01 0.01; visual mesh filename=package://chessbot_robot/meshes/irb140/visual/link_5.stl scale=0.01 0.01 0.01
- added link link_6, mass 1.0; collision mesh filename=package://chessbot_robot/meshes/irb140/collision/link_6.stl scale=0.01 0.01 0.01; visual mesh filename=package://chessbot_robot/meshes/irb140/visual/link_6.stl scale=0.01 0.01 0.01
- added link tool0
- added link world
Joints:
- added joint base_link-base: type fixed, parent base_link, child base, origin xyz=0 0 0 rpy=0 0 0
- added joint camera_joint: type fixed, parent link_6, child camera_link, origin xyz=0 0 0 rpy=0 0 0
- added joint fixed: type fixed, parent map, child base_link
- added joint joint_1: type revolute, parent base_link, child link_1, origin xyz=0 0 0 rpy=0 0 0, axis 0 0 1, limit lower=-3.1416 upper=3.1416 effort=0 velocity=2.618
- added joint joint_2: type revolute, parent link_1, child link_2, origin xyz=0.070 0 0.352 rpy=0 0 0, axis 0 1 0, limit lower=-1.7453 upper=1.7453 effort=0 velocity=2.618
- added joint joint_3: type revolute, parent link_2, child link_3, origin xyz=0 -0.065 0.360 rpy=0 0 0, axis 0 1 0, limit lower=-2.4434 upper=2.4434 effort=0 velocity=2.618
- added joint joint_4: type revolute, parent link_3, child link_4, origin xyz=0.239 0.065 0 rpy=0 0 0, axis 1 0 0, limit lower=-3.49 upper=3.49 effort=0 velocity=6.2832
- added joint joint_5: type revolute, parent link_4, child link_5, origin xyz=0.141 0 0 rpy=0 0 0, axis 0 1 0, limit lower=-2.0071 upper=2.0071 effort=0 velocity=6.2832
- added joint joint_6: type revolute, parent link_5, child link_6, origin xyz=0.065 0 0 rpy=0 0 0, axis 1 0 0, limit lower=-6.9813 upper=6.9813 effort=0 velocity=7.854
- added joint joint_6-tool0: type fixed, parent link_6, child tool0, origin xyz=0 0 0 rpy=0 0 0

Commit message: Sensor update and actuators definition. No controllers

File: chessbot_ws/src/chessbot_robot/urdf/irb140.xacro (robot description, xacro)
@@ -4,5 +4,5 @@
 	<xacro:include filename="$(find chessbot_robot)/urdf/gazebo/camera_sensor.gazebo"/>
 	<gazebo>
-    	<static>true</static>
+    	<static>false</static>
 	</gazebo>
 </robot>

File: chessbot_ws/src/chessbot_robot/urdf/robot/irb140_robot.xacro (robot description, xacro)
@@ -3,4 +3,6 @@
   <xacro:include filename="$(find chessbot_robot)/urdf/robot/links.xacro"/>
   <xacro:include filename="$(find chessbot_robot)/urdf/robot/joints.xacro"/>
-  <static>true</static>
+  <xacro:include filename="$(find chessbot_robot)/urdf/robot/actuators.xacro"/>
+  <!-- TODO: moverl los motores del robot  -->
+  <static>false</static>
 </robot>

File: chessbot_ws/src/chessbot_robot/urdf/robot/links.xacro (robot description, xacro)
@@ -9,7 +9,4 @@
         <mesh filename="package://chessbot_robot/meshes/irb140/visual/base_link.stl" scale="0.01 0.01 0.01"/>
       </geometry>
-      <material name="abb_orange">
-        <color rgba="1 0.43 0 1"/>
-      </material>
     </visual>
     <collision>
@@ -24,5 +21,5 @@
       <origin xyz="0.0 0.0 0.0" rpy="0.0 0.0 0.0"/>
       <mass value="1.0"/>
-      <inertia ixx="0.0" ixy="0.0" ixz="0.0" iyy="0.0" iyz="0.0" izz="0.0"/>
+      <inertia ixx="1.0" ixy="1.0" ixz="1.0" iyy="1.0" iyz="1.0" izz="1.0"/>
     </inertial>
   </link>
@@ -45,5 +42,5 @@
       <origin xyz="0.0 0.0 0.0" rpy="0.0 0.0 0.0"/>
       <mass value="1.0"/>
-      <inertia ixx="0.0" ixy="0.0" ixz="0.0" iyy="0.0" iyz="0.0" izz="0.0"/>
+      <inertia ixx="1.0" ixy="1.0" ixz="1.0" iyy="1.0" iyz="1.0" izz="1.0"/>
     </inertial>
   </link>
@@ -54,5 +51,5 @@
         <mesh filename="package://chessbot_robot/meshes/irb140/visual/link_2.stl" scale="0.01 0.01 0.01"/>
       </geometry>
-      <material name="abb_orange"/>
+      <!-- <material name="abb_orange"/> -->
     </visual>
     <collision>
@@ -66,5 +63,5 @@
       <origin xyz="0.0 0.0 0.0" rpy="0.0 0.0 0.0"/>
       <mass value="1.0"/>
-      <inertia ixx="0.0" ixy="0.0" ixz="0.0" iyy="0.0" iyz="0.0" izz="0.0"/>
+      <inertia ixx="1.0" ixy="1.0" ixz="1.0" iyy="1.0" iyz="1.0" izz="1.0"/>
     </inertial>
   </link>
@@ -87,5 +84,5 @@
       <origin xyz="0.0 0.0 0.0" rpy="0.0 0.0 0.0"/>
       <mass value="1.0"/>
-      <inertia ixx="0.0" ixy="0.0" ixz="0.0" iyy="0.0" iyz="0.0" izz="0.0"/>
+      <inertia ixx="1.0" ixy="1.0" ixz="1.0" iyy="1.0" iyz="1.0" izz="1.0"/>
     </inertial>
   </link>
@@ -108,5 +105,5 @@
       <origin xyz="0.0 0.0 0.0" rpy="0.0 0.0 0.0"/>
       <mass value="1.0"/>
-      <inertia ixx="0.0" ixy="0.0" ixz="0.0" iyy="0.0" iyz="0.0" izz="0.0"/>
+      <inertia ixx="1.0" ixy="1.0" ixz="1.0" iyy="1.0" iyz="1.0" izz="1.0"/>
     </inertial>
   </link>
@@ -129,5 +126,5 @@
       <origin xyz="0.0 0.0 0.0" rpy="0.0 0.0 0.0"/>
       <mass value="1.0"/>
-      <inertia ixx="0.0" ixy="0.0" ixz="0.0" iyy="0.0" iyz="0.0" izz="0.0"/>
+      <inertia ixx="1.0" ixy="1.0" ixz="1.0" iyy="1.0" iyz="1.0" izz="1.0"/>
     </inertial>
   </link>
@@ -150,5 +147,5 @@
       <origin xyz="0.0 0.0 0.0" rpy="0.0 0.0 0.0"/>
       <mass value="1.0"/>
-      <inertia ixx="0.0" ixy="0.0" ixz="0.0" iyy="0.0" iyz="0.0" izz="0.0"/>
+      <inertia ixx="1.0" ixy="1.0" ixz="1.0" iyy="1.0" iyz="1.0" izz="1.0"/>
     </inertial>
   </link>
@@ -157,10 +154,11 @@
       <origin xyz="0.0 0.0 0.0" rpy="0.0 0.0 0.0"/>
       <mass value="0.0"/>
-      <inertia ixx="0.0" ixy="0.0" ixz="0.0" iyy="0.0" iyz="0.0" izz="0.0"/>
+      <inertia ixx="1.0" ixy="1.0" ixz="1.0" iyy="1.0" iyz="1.0" izz="1.0"/>
     </inertial>
     <visual name="">
       <origin xyz="0.0 0.0 0.0" rpy="0.0 0.0 0.0"/>
       <geometry>
-        <box size="0.1 0.1 0.1"/>
+        <!-- TODO: Replace with a camera model stl  -->
+        <box size="0.06 0.1 0.06"/>
       </geometry>
       <material name="">
@@ -172,5 +170,6 @@
       <origin xyz="0.0 0.0 0.0" rpy="0.0 0.0 0.0"/>
       <geometry>
-        <box size="0.0 0.0 0.0"/>
+        <!-- TODO: Replace with a camera model stl  -->
+        <box size="0.06 0.1 0.06"/>
       </geometry>
     </collision>
